File: schematics/receiver/rfm95/receiver_rfm95.sch (EAGLE design)
At the start: 47 parts, among them IC1 ATMEGA328P, Q1 16MHz, Q2 BC817-16SMD, U2 AMS1117_3.3, U3 RA-02_LORA_MODULE

Commit message: Enhancements: ST7920 LCD Support, Documentation and schematics updates, minor fixes and improvements. (#51)
* Update readme.md

* Delete assets/Bm437_Portfolio_6x8_modBUK.FON

* Add files via upload

* Update readme.txt

* Update readme.txt

* Add files via upload

* Delete schematics directory

* Add files via upload

* Update config.h

Added support for ST7920 based LCD.

* Update font.cpp

Added support for ST7920 based LCD.

* Update ui_128x64.cpp

- Added support for ST7920 based LCD.
- Fixed minor bug in when showing tool-tip in mixer monitor screen, when the output is none.
- Other minor improvements.

* Update sdStore.cpp

- Added support for ST7920 LCD.
- Other minor improvements.

* Update font.h

Added support for ST7920 LCD.

* Update ui.h

Added support for ST7920 LCD.

* Add files via upload

Added support for ST7920 LCD.

* Update config.h

* Update receiver.cpp

* Update rfComm.cpp

* Add files via upload

* Update README.md

* Update config.h

Bump version number.

* Add files via upload
Parts:
- removed U3: RA-02_LORA_MODULE, RA-02_Lora_module:RA-02_LORA_MODULE
- added U1: RFM95_LORA_MODULE, RFM95_Lora_module:RFM95_LORA_MODULE
- R10, R11, R12, R16, R17, R7, R9: value 4.7k -> 5.6k
- R4, R5, R6, R8: value 4.7k -> 10k
Connections:
- removed net N$5: PAD1.P, U3.GND
- new net N$17: PAD1.P, U1.ANT
- net +3V3: now also U1.3.3V; no longer U3.3.3V
- net GND: now also U1.GND, U1.GND@1, U1.GND@2; no longer U3.GND@2, U3.GND@3, U3.GND@4
- net N$11: now also U1.MISO; no longer U3.MISO
- net N$6: now also U1.RESET; no longer U3.RESET
- net N$7: now also U1.NSS; no longer U3.NSS
- net N$8: now also U1.SCK; no longer U3.SCK
- net N$9: now also U1.MOSI; no longer U3.MOSI
Other:
- moved on the sheet: J2, J3, J4, J6, JP1, PAD1, R16, R17, R18, R19, R20, R21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
