File: schematics/receiver/rfm95/receiver_mini_rfm95.brd (EAGLE design)
At the start: 20 x 26 mm, 23 parts, among them IC1 ATMEGA328P, Q1 16MHz, U1 RFM95_LORA_MODULE, U2 AMS1117_3.3

Commit message: Fixed incorrect resistor values
- Fixed incorrect resistor values in the level shifters.
Parts:
- R10, R11, R8, R9: value 5.6k -> 560
- R3, R4, R5, R6: value 10k -> 1k
- R7: value 5.6k -> 1k
Changed lines of the file:
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@@
 <attribute name="VALUE" x="4.595" y="4.575" size="1.27" layer="27"/>
 </element>
-<element name="R7" library="rcl" package="R0805" value="5.6k" x="2.25" y="3.5" smashed="yes" rot="R270">
+<element name="R7" library="rcl" package="R0805" value="1k" x="2.25" y="3.5" smashed="yes" rot="R270">
 <attribute name="NAME" x="3.2025" y="1.2775" size="1.27" layer="25" rot="R270" display="off"/>
 <attribute name="VALUE" x="-0.29" y="4.135" size="1.27" layer="27" rot="R270"/>
@@
 <attribute name="VALUE" x="16.365" y="9.71" size="1.27" layer="27"/>
 </element>
-<element name="R9" library="rcl" package="R0805" value="5.6k" x="2.25" y="11" smashed="yes">
+<element name="R9" library="rcl" package="R0805" value="560" x="2.25" y="11" smashed="yes">
 <attribute name="NAME" x="1.615" y="12.27" size="1.27" layer="25" display="off"/>
 <attribute name="VALUE" x="1.615" y="8.46" size="1.27" layer="27"/>
 </element>
-<element name="R5" library="rcl" package="R0805" value="10k" x="2.25" y="16.75" smashed="yes">
+<element name="R5" library="rcl" package="R0805" value="1k" x="2.25" y="16.75" smashed="yes">
 <attribute name="NAME" x="-3.1475" y="16.115" size="1.27" layer="25" display="off"/>
 <attribute name="VALUE" x="1.615" y="14.21" size="1.27" layer="27"/>
 </element>
-<element name="R8" library="rcl" package="R0805" value="5.6k" x="6.75" y="22.75" smashed="yes" rot="R270">
+<element name="R8" library="rcl" package="R0805" value="560" x="6.75" y="22.75" smashed="yes" rot="R270">
 <attribute name="NAME" x="8.02" y="23.385" size="1.27" layer="25" rot="R270" display="off"/>
 <attribute name="VALUE" x="4.21" y="23.385" size="1.27" layer="27" rot="R270"/>
 </element>
-<element name="R4" library="rcl" package="R0805" value="10k" x="2.25" y="13.25" smashed="yes">
+<element name="R4" library="rcl" package="R0805" value="1k" x="2.25" y="13.25" smashed="yes">
 <attribute name="NAME" x="-3.1475" y="12.615" size="1.27" layer="25" display="off"/>
 <attribute name="VALUE" x="1.615" y="10.71" size="1.27" layer="27"/>
 </element>
-<element name="R10" library="rcl" package="R0805" value="5.6k" x="2.25" y="19" smashed="yes">
+<element name="R10" library="rcl" package="R0805" value="560" x="2.25" y="19" smashed="yes">
 <attribute name="NAME" x="-3.465" y="13.92" size="1.27" layer="25" display="off"/>
 <attribute name="VALUE" x="1.615" y="16.46" size="1.27" layer="27"/>
 </element>
-<element name="R3" library="rcl" package="R0805" value="10k" x="4.5" y="22.75" smashed="yes" rot="R270">
+<element name="R3" library="rcl" package="R0805" value="1k" x="4.5" y="22.75" smashed="yes" rot="R270">
 <attribute name="NAME" x="3.865" y="28.1475" size="1.27" layer="25" rot="R270" display="off"/>
 <attribute name="VALUE" x="1.96" y="23.385" size="1.27" layer="27" rot="R270"/>
 </element>
-<element name="R11" library="rcl" package="R0805" value="5.6k" x="2.25" y="8.75" smashed="yes">
+<element name="R11" library="rcl" package="R0805" value="560" x="2.25" y="8.75" smashed="yes">
 <attribute name="NAME" x="1.615" y="10.02" size="1.27" layer="25" display="off"/>
 <attribute name="VALUE" x="1.615" y="6.21" size="1.27" layer="27"/>
 </element>
-<element name="R6" library="rcl" package="R0805" value="10k" x="2.25" y="6.5" smashed="yes">
+<element name="R6" library="rcl" package="R0805" value="1k" x="2.25" y="6.5" smashed="yes">
 <attribute name="NAME" x="-4.4175" y="5.865" size="1.27" layer="25" display="off"/>
 <attribute name="VALUE" x="1.615" y="3.96" size="1.27" layer="27"/>
