File: schematics/receiver/rfm95/receiver_rfm95.brd (EAGLE design)
At the start: 29.8 x 34.9 mm, 47 parts, among them IC1 ATMEGA328P, Q1 16MHz, U1 RFM95_LORA_MODULE, U2 AMS1117_3.3

Commit message: Fixed incorrect resistor values
- Fixed incorrect resistor values in the level shifters.
Parts:
- R10, R11, R12, R9: value 5.6k -> 560
- R4, R5, R6, R8: value 10k -> 1k
- R7: value 5.6k -> 1k
Changed lines of the file:
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@@
 <attribute name="VALUE" x="22.5425" y="23.97125" size="1.27" layer="28" rot="MR180"/>
 </element>
-<element name="R9" library="rcl" package="R0805" value="5.6k" x="4.7625" y="23.1775" smashed="yes" rot="MR180">
+<element name="R9" library="rcl" package="R0805" value="560" x="4.7625" y="23.1775" smashed="yes" rot="MR180">
 <attribute name="NAME" x="0.3175" y="23.8125" size="1.016" layer="26" ratio="15" rot="MR180" display="off"/>
 <attribute name="VALUE" x="4.1275" y="25.7175" size="1.27" layer="28" rot="MR180"/>
 </element>
-<element name="R10" library="rcl" package="R0805" value="5.6k" x="4.7625" y="25.0825" smashed="yes" rot="MR180">
+<element name="R10" library="rcl" package="R0805" value="560" x="4.7625" y="25.0825" smashed="yes" rot="MR180">
 <attribute name="NAME" x="0" y="25.7175" size="1.016" layer="26" ratio="15" rot="MR180" display="off"/>
 <attribute name="VALUE" x="4.1275" y="27.6225" size="1.27" layer="28" rot="MR180"/>
 </element>
-<element name="R11" library="rcl" package="R0805" value="5.6k" x="4.7625" y="28.8925" smashed="yes" rot="MR180">
+<element name="R11" library="rcl" package="R0805" value="560" x="4.7625" y="28.8925" smashed="yes" rot="MR180">
 <attribute name="NAME" x="0" y="29.5275" size="1.016" layer="26" ratio="15" rot="MR180" display="off"/>
 <attribute name="VALUE" x="4.1275" y="31.4325" size="1.27" layer="28" rot="MR180"/>
 </element>
-<element name="R12" library="rcl" package="R0805" value="5.6k" x="4.7625" y="26.9875" smashed="yes" rot="MR180">
+<element name="R12" library="rcl" package="R0805" value="560" x="4.7625" y="26.9875" smashed="yes" rot="MR180">
 <attribute name="NAME" x="0" y="27.6225" size="1.016" layer="26" ratio="15" rot="MR180" display="off"/>
 <attribute name="VALUE" x="4.1275" y="29.5275" size="1.27" layer="28" rot="MR180"/>
 </element>
-<element name="R8" library="rcl" package="R0805" value="10k" x="24.13" y="21.2725" smashed="yes" rot="R90">
+<element name="R8" library="rcl" package="R0805" value="1k" x="24.13" y="21.2725" smashed="yes" rot="R90">
 <attribute name="NAME" x="19.3675" y="22.225" size="1.016" layer="25" ratio="15" rot="SR270" display="off"/>
 <attribute name="VALUE" x="26.67" y="20.6375" size="1.27" layer="27" rot="R90"/>
 </element>
-<element name="R6" library="rcl" package="R0805" value="10k" x="24.13" y="25.0825" smashed="yes" rot="R90">
+<element name="R6" library="rcl" package="R0805" value="1k" x="24.13" y="25.0825" smashed="yes" rot="R90">
 <attribute name="NAME" x="19.3675" y="26.035" size="1.016" layer="25" ratio="15" rot="SR270" display="off"/>
 <attribute name="VALUE" x="26.67" y="24.4475" size="1.27" layer="27" rot="R90"/>
 </element>
-<element name="R5" library="rcl" package="R0805" value="10k" x="24.13" y="28.8925" smashed="yes" rot="R270">
+<element name="R5" library="rcl" package="R0805" value="1k" x="24.13" y="28.8925" smashed="yes" rot="R270">
 <attribute name="NAME" x="19.685" y="29.5275" size="1.016" layer="25" ratio="15" rot="SR270" display="off"/>
 <attribute name="VALUE" x="21.59" y="29.5275" size="1.27" layer="27" rot="R270"/>
 </element>
-<element name="R4" library="rcl" package="R0805" value="10k" x="24.13" y="32.7025" smashed="yes" rot="R270">
+<element name="R4" library="rcl" package="R0805" value="1k" x="24.13" y="32.7025" smashed="yes" rot="R270">
 <attribute name="NAME" x="19.685" y="33.655" size="1.016" layer="25" ratio="15" rot="SR270" display="off"/>
 <attribute name="VALUE" x="21.59" y="33.3375" size="1.27" layer="27" rot="R270"/>
@@
 <attribute name="VALUE" x="13.6525" y="12.065" size="1.27" layer="27"/>
 </element>
-<element name="R7" library="rcl" package="R0805" value="5.6k" x="19.685" y="11.1125" smashed="yes" rot="R270">
+<element name="R7" library="rcl" package="R0805" value="1k" x="19.685" y="11.1125" smashed="yes" rot="R270">
 <attribute name="NAME" x="20.32" y="9.2075" size="1.016" layer="25" ratio="15" rot="SR180" display="off"/>
 <attribute name="VALUE" x="17.145" y="11.7475" size="1.27" layer="27" rot="R270"/>
