File: schematics/transmitter/secondary/stx_v2.brd (EAGLE design)
At the start: 27.9 x 47 mm, 29 parts, among them Q3 16MHz, T1 BC337, U1 ATMEGA328P_PDIP, U2 AMS1117_3.3

Commit message: Fixed incorrect resistor values.
- Fixed incorrect resistor values in the level shifters. 
- Fixed a mistake in the silk screen where the R4 and R9 label positions where swapped.
Parts:
- R10, R11, R12, R9: value 5.6k -> 560
- R4, R5, R6, R8: value 10k -> 1k
- R7: value 5.6k -> 1k
Changed lines of the file:
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@@
 <attribute name="VALUE" x="8.6106" y="33.5026" size="0.9906" layer="27" ratio="10" rot="R180"/>
 </element>
-<element name="R9" library="rcl" package="0204V" value="5.6k" x="24.13" y="10.16" smashed="yes" rot="R270">
-<attribute name="NAME" x="26.035" y="9.36625" size="1.016" layer="25" ratio="15" rot="R90"/>
+<element name="R9" library="rcl" package="0204V" value="560" x="24.13" y="10.16" smashed="yes" rot="R270">
+<attribute name="NAME" x="23.495" y="9.36625" size="1.016" layer="25" ratio="15" rot="R90"/>
 <attribute name="VALUE" x="21.8186" y="12.2936" size="1.27" layer="27" ratio="10" rot="R270"/>
 </element>
-<element name="R10" library="rcl" package="0204V" value="5.6k" x="24.13" y="35.56" smashed="yes" rot="R270">
+<element name="R10" library="rcl" package="0204V" value="560" x="24.13" y="35.56" smashed="yes" rot="R270">
 <attribute name="NAME" x="23.33625" y="34.44875" size="1.016" layer="25" ratio="15" rot="R90"/>
 <attribute name="VALUE" x="21.8186" y="37.6936" size="1.27" layer="27" ratio="10" rot="R270"/>
 </element>
-<element name="R11" library="rcl" package="0204V" value="5.6k" x="24.13" y="25.4" smashed="yes" rot="R270">
+<element name="R11" library="rcl" package="0204V" value="560" x="24.13" y="25.4" smashed="yes" rot="R270">
 <attribute name="NAME" x="23.33625" y="24.13" size="1.016" layer="25" ratio="15" rot="R90"/>
 <attribute name="VALUE" x="21.8186" y="27.5336" size="1.27" layer="27" ratio="10" rot="R270"/>
 </element>
-<element name="R12" library="rcl" package="0204V" value="5.6k" x="24.13" y="15.24" smashed="yes" rot="R270">
+<element name="R12" library="rcl" package="0204V" value="560" x="24.13" y="15.24" smashed="yes" rot="R270">
 <attribute name="NAME" x="26.035" y="13.97" size="1.016" layer="25" ratio="15" rot="R90"/>
 <attribute name="VALUE" x="21.8186" y="17.3736" size="1.27" layer="27" ratio="10" rot="R270"/>
 </element>
-<element name="R8" library="rcl" package="0204V" value="10k" x="24.13" y="20.32" smashed="yes" rot="R270">
+<element name="R8" library="rcl" package="0204V" value="1k" x="24.13" y="20.32" smashed="yes" rot="R270">
 <attribute name="NAME" x="23.33625" y="19.685" size="1.016" layer="25" ratio="15" rot="R90"/>
 <attribute name="VALUE" x="21.8186" y="22.4536" size="1.27" layer="27" ratio="10" rot="R270"/>
 </element>
-<element name="R6" library="rcl" package="0204V" value="10k" x="24.13" y="30.48" smashed="yes" rot="R270">
+<element name="R6" library="rcl" package="0204V" value="1k" x="24.13" y="30.48" smashed="yes" rot="R270">
 <attribute name="NAME" x="23.33625" y="29.68625" size="1.016" layer="25" ratio="15" rot="R90"/>
 <attribute name="VALUE" x="21.8186" y="32.6136" size="1.27" layer="27" ratio="10" rot="R270"/>
 </element>
-<element name="R5" library="rcl" package="0204V" value="10k" x="24.13" y="39.84625" smashed="yes" rot="R270">
+<element name="R5" library="rcl" package="0204V" value="1k" x="24.13" y="39.84625" smashed="yes" rot="R270">
 <attribute name="NAME" x="23.33625" y="39.0525" size="1.016" layer="25" ratio="15" rot="R90"/>
 <attribute name="VALUE" x="21.8186" y="41.97985" size="1.27" layer="27" ratio="10" rot="R270"/>
 </element>
-<element name="R4" library="rcl" package="0204V" value="10k" x="26.67" y="10.16" smashed="yes" rot="R90">
-<attribute name="NAME" x="23.495" y="9.36625" size="1.016" layer="25" ratio="15" rot="R90"/>
+<element name="R4" library="rcl" package="0204V" value="1k" x="26.67" y="10.16" smashed="yes" rot="R90">
+<attribute name="NAME" x="26.035" y="9.36625" size="1.016" layer="25" ratio="15" rot="R90"/>
 <attribute name="VALUE" x="28.9814" y="8.0264" size="1.27" layer="27" ratio="10" rot="R90"/>
 </element>
-<element name="R7" library="rcl" package="0204V" value="5.6k" x="25.4" y="6.35" smashed="yes" rot="R180">
+<element name="R7" library="rcl" package="0204V" value="1k" x="25.4" y="6.35" smashed="yes" rot="R180">
 <attribute name="NAME" x="26.51125" y="7.9375" size="1.016" layer="25" ratio="15" rot="R180"/>
 <attribute name="VALUE" x="27.5336" y="8.6614" size="1.27" layer="27" ratio="10" rot="R180"/>
