File: schematics/transmitter/secondary/stx_v2.sch (EAGLE design)
At the start: 29 parts, among them Q3 16MHz, T1 BC337, U1 ATMEGA328P_PDIP, U2 AMS1117_3.3

Commit message: Fixed incorrect resistor values.
- Fixed incorrect resistor values in the level shifters. 
- Fixed a mistake in the silk screen where the R4 and R9 label positions where swapped.
Parts:
- R10, R11, R12, R9: value 5.6k -> 560
- R4, R5, R6, R8: value 10k -> 1k
- R7: value 5.6k -> 1k
Changed lines of the file:
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@@
 <part name="P+9" library="supply1" deviceset="+5V" device=""/>
 <part name="P+4" library="supply1" deviceset="+5V" device=""/>
-<part name="R9" library="rcl" deviceset="R-US_" device="0204/2V" value="5.6k"/>
-<part name="R10" library="rcl" deviceset="R-US_" device="0204/2V" value="5.6k"/>
-<part name="R11" library="rcl" deviceset="R-US_" device="0204/2V" value="5.6k"/>
-<part name="R12" library="rcl" deviceset="R-US_" device="0204/2V" value="5.6k"/>
-<part name="R8" library="rcl" deviceset="R-US_" device="0204/2V" value="10k"/>
-<part name="R6" library="rcl" deviceset="R-US_" device="0204/2V" value="10k"/>
-<part name="R5" library="rcl" deviceset="R-US_" device="0204/2V" value="10k"/>
-<part name="R4" library="rcl" deviceset="R-US_" device="0204/2V" value="10k"/>
+<part name="R9" library="rcl" deviceset="R-US_" device="0204/2V" value="560"/>
+<part name="R10" library="rcl" deviceset="R-US_" device="0204/2V" value="560"/>
+<part name="R11" library="rcl" deviceset="R-US_" device="0204/2V" value="560"/>
+<part name="R12" library="rcl" deviceset="R-US_" device="0204/2V" value="560"/>
+<part name="R8" library="rcl" deviceset="R-US_" device="0204/2V" value="1k"/>
+<part name="R6" library="rcl" deviceset="R-US_" device="0204/2V" value="1k"/>
+<part name="R5" library="rcl" deviceset="R-US_" device="0204/2V" value="1k"/>
+<part name="R4" library="rcl" deviceset="R-US_" device="0204/2V" value="1k"/>
 <part name="GND8" library="supply1" deviceset="GND" device=""/>
-<part name="R7" library="rcl" deviceset="R-US_" device="0204/2V" value="5.6k"/>
+<part name="R7" library="rcl" deviceset="R-US_" device="0204/2V" value="1k"/>
 <part name="R2" library="rcl" deviceset="R-US_" device="0204/7" value="10k"/>
 <part name="+3V32" library="supply1" deviceset="+3V3" device=""/>
@@
 </instance>
 <instance part="R7" gate="G$1" x="93.98" y="-35.56" smashed="yes">
-<attribute name="NAME" x="91.694" y="-34.3154" size="1.778" layer="95"/>
-<attribute name="VALUE" x="90.17" y="-38.862" size="1.778" layer="96"/>
+<attribute name="NAME" x="92.71" y="-34.0614" size="1.778" layer="95"/>
+<attribute name="VALUE" x="92.71" y="-38.862" size="1.778" layer="96"/>
 </instance>
 <instance part="R2" gate="G$1" x="76.2" y="-35.56" smashed="yes">
-<attribute name="NAME" x="80.01" y="-37.8714" size="1.778" layer="95"/>
-<attribute name="VALUE" x="72.39" y="-38.862" size="1.778" layer="96"/>
+<attribute name="NAME" x="74.676" y="-34.0614" size="1.778" layer="95"/>
+<attribute name="VALUE" x="73.914" y="-38.862" size="1.778" layer="96"/>
 </instance>
 <instance part="+3V32" gate="G$1" x="66.04" y="-35.56" smashed="yes" rot="R90">
@@
 <attribute name="VALUE" x="20.32" y="33.02" size="1.778" layer="96" rot="R270"/>
 </instance>
-<instance part="T1" gate="G$1" x="83.82" y="-38.1" rot="R270"/>
+<instance part="T1" gate="G$1" x="83.82" y="-38.1" smashed="yes" rot="R270">
+<attribute name="NAME" x="81.28" y="-43.18" size="1.778" layer="95"/>
+<attribute name="VALUE" x="81.28" y="-45.72" size="1.778" layer="96"/>
+</instance>
 <instance part="J6" gate="G$1" x="157.48" y="30.48" rot="R180"/>
 <instance part="D2" gate="G$1" x="83.82" y="104.14" rot="R90"/>
