File: schematics/receiver/ra02/receiver_mini_ra02.sch (EAGLE design)
At the start: 23 parts, among them IC1 ATMEGA328P, Q1 16MHz, Q2 BC817-16SMD, U2 AMS1117_3.3, U3 RA-02_LORA_MODULE

Commit message: Fixed incorrect resistor values.
- Fixed incorrect resistor values in the level shifters.
Parts:
- R10, R11, R8, R9: value 4.7k -> 560
- R3, R4, R5, R6: value 10k -> 1k
- R7: value 4.7k -> 1k
Changed lines of the file:
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@@
 <part name="C3" library="rcl" deviceset="C-EU" device="C0805K" value="100n"/>
 <part name="Q2" library="transistor-npn" deviceset="BC817*" device="SMD" technology="-16" value=""/>
-<part name="R7" library="rcl" deviceset="R-US_" device="R0805" value="4.7k"/>
+<part name="R7" library="rcl" deviceset="R-US_" device="R0805" value="1k"/>
 <part name="R2" library="rcl" deviceset="R-US_" device="R0805" value="10k"/>
 <part name="+3V32" library="supply1" deviceset="+3V3" device=""/>
@@
 <part name="R12" library="rcl" deviceset="R-US_" device="R0805" value="1k"/>
 <part name="P+4" library="supply1" deviceset="+5V" device=""/>
-<part name="R9" library="rcl" deviceset="R-US_" device="R0805" value="4.7k"/>
-<part name="R5" library="rcl" deviceset="R-US_" device="R0805" value="10k"/>
-<part name="R8" library="rcl" deviceset="R-US_" device="R0805" value="4.7k"/>
-<part name="R4" library="rcl" deviceset="R-US_" device="R0805" value="10k"/>
-<part name="R10" library="rcl" deviceset="R-US_" device="R0805" value="4.7k"/>
-<part name="R3" library="rcl" deviceset="R-US_" device="R0805" value="10k"/>
-<part name="R11" library="rcl" deviceset="R-US_" device="R0805" value="4.7k"/>
-<part name="R6" library="rcl" deviceset="R-US_" device="R0805" value="10k"/>
+<part name="R9" library="rcl" deviceset="R-US_" device="R0805" value="560"/>
+<part name="R5" library="rcl" deviceset="R-US_" device="R0805" value="1k"/>
+<part name="R8" library="rcl" deviceset="R-US_" device="R0805" value="560"/>
+<part name="R4" library="rcl" deviceset="R-US_" device="R0805" value="1k"/>
+<part name="R10" library="rcl" deviceset="R-US_" device="R0805" value="560"/>
+<part name="R3" library="rcl" deviceset="R-US_" device="R0805" value="1k"/>
+<part name="R11" library="rcl" deviceset="R-US_" device="R0805" value="560"/>
+<part name="R6" library="rcl" deviceset="R-US_" device="R0805" value="1k"/>
 <part name="GND7" library="supply1" deviceset="GND" device=""/>
 <part name="P+2" library="supply1" deviceset="+5V" device=""/>
