File: schematics/receiver/receiver_v2.brd (EAGLE design)
At the start: 40.6 x 59.7 mm, 51 parts, among them Q3 16MHz, T1 BC337, U1 ATMEGA328P_PDIP, U2 AMS1117_3.3

Commit message: Fixed incorrect resistor values
- Fixed incorrect resistor values in the level shifters.
Parts:
- R10, R11, R12, R9: value 5.6k -> 560
- R4, R5, R6, R8: value 10k -> 1k
- R7: value 5.6k -> 1k
Changed lines of the file:
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@@
 <attribute name="VALUE" x="14.9606" y="48.7426" size="0.9906" layer="27" ratio="10" rot="R180"/>
 </element>
-<element name="R9" library="rcl" package="0204V" value="5.6k" x="30.48" y="27.94" smashed="yes" rot="R270">
+<element name="R9" library="rcl" package="0204V" value="560" x="30.48" y="27.94" smashed="yes" rot="R270">
 <attribute name="NAME" x="32.22625" y="26.82875" size="1.016" layer="25" ratio="15" rot="R90"/>
 <attribute name="VALUE" x="28.1686" y="30.0736" size="1.27" layer="27" ratio="10" rot="R270"/>
 </element>
-<element name="R10" library="rcl" package="0204V" value="5.6k" x="33.02" y="27.94" smashed="yes" rot="R270">
+<element name="R10" library="rcl" package="0204V" value="560" x="33.02" y="27.94" smashed="yes" rot="R270">
 <attribute name="NAME" x="34.76625" y="26.82875" size="1.016" layer="25" ratio="15" rot="R90"/>
 <attribute name="VALUE" x="30.7086" y="30.0736" size="1.27" layer="27" ratio="10" rot="R270"/>
 </element>
-<element name="R11" library="rcl" package="0204V" value="5.6k" x="38.1" y="27.94" smashed="yes" rot="R270">
+<element name="R11" library="rcl" package="0204V" value="560" x="38.1" y="27.94" smashed="yes" rot="R270">
 <attribute name="NAME" x="40.005" y="26.82875" size="1.016" layer="25" ratio="15" rot="R90"/>
 <attribute name="VALUE" x="35.7886" y="30.0736" size="1.27" layer="27" ratio="10" rot="R270"/>
 </element>
-<element name="R12" library="rcl" package="0204V" value="5.6k" x="35.56" y="27.94" smashed="yes" rot="R270">
+<element name="R12" library="rcl" package="0204V" value="560" x="35.56" y="27.94" smashed="yes" rot="R270">
 <attribute name="NAME" x="37.30625" y="26.82875" size="1.016" layer="25" ratio="15" rot="R90"/>
 <attribute name="VALUE" x="33.2486" y="30.0736" size="1.27" layer="27" ratio="10" rot="R270"/>
 </element>
-<element name="R8" library="rcl" package="0204V" value="10k" x="35.56" y="33.02" smashed="yes" rot="R270">
+<element name="R8" library="rcl" package="0204V" value="1k" x="35.56" y="33.02" smashed="yes" rot="R270">
 <attribute name="NAME" x="37.30625" y="32.22625" size="1.016" layer="25" ratio="15" rot="R90"/>
 <attribute name="VALUE" x="33.2486" y="35.1536" size="1.27" layer="27" ratio="10" rot="R270"/>
 </element>
-<element name="R6" library="rcl" package="0204V" value="10k" x="38.1" y="33.02" smashed="yes" rot="R270">
+<element name="R6" library="rcl" package="0204V" value="1k" x="38.1" y="33.02" smashed="yes" rot="R270">
 <attribute name="NAME" x="39.84625" y="32.22625" size="1.016" layer="25" ratio="15" rot="R90"/>
 <attribute name="VALUE" x="35.7886" y="35.1536" size="1.27" layer="27" ratio="10" rot="R270"/>
 </element>
-<element name="R5" library="rcl" package="0204V" value="10k" x="33.02" y="33.02" smashed="yes" rot="R270">
+<element name="R5" library="rcl" package="0204V" value="1k" x="33.02" y="33.02" smashed="yes" rot="R270">
 <attribute name="NAME" x="34.76625" y="32.22625" size="1.016" layer="25" ratio="15" rot="R90"/>
 <attribute name="VALUE" x="30.7086" y="35.1536" size="1.27" layer="27" ratio="10" rot="R270"/>
 </element>
-<element name="R4" library="rcl" package="0204V" value="10k" x="30.48" y="33.02" smashed="yes" rot="R270">
+<element name="R4" library="rcl" package="0204V" value="1k" x="30.48" y="33.02" smashed="yes" rot="R270">
 <attribute name="NAME" x="32.22625" y="32.22625" size="1.016" layer="25" ratio="15" rot="R90"/>
 <attribute name="VALUE" x="28.1686" y="35.1536" size="1.27" layer="27" ratio="10" rot="R270"/>
 </element>
-<element name="R7" library="rcl" package="0204V" value="5.6k" x="30.48" y="22.86" smashed="yes" rot="R90">
+<element name="R7" library="rcl" package="0204V" value="1k" x="30.48" y="22.86" smashed="yes" rot="R90">
 <attribute name="NAME" x="32.22625" y="22.06625" size="1.016" layer="25" ratio="15" rot="R90"/>
 <attribute name="VALUE" x="32.7914" y="20.7264" size="1.27" layer="27" ratio="10" rot="R90"/>
